File: hardware/IO.sch (KiCad schematic (older format))
At the start: 0 parts

Commit message: Pcb development (#1)
* PCB Finished and Ordered
Parts:
- added J1: Conn_02x04_Odd_Even, Pin_Headers:Pin_Header_Straight_2x04_Pitch2.54mm, symbol Connector_Generic:Conn_02x04_Odd_Even
- added J2: Conn_01x12, Pin_Headers:Pin_Header_Straight_2x06_Pitch2.54mm, symbol Connector_Generic:Conn_01x12
- added J3: Conn_02x03_Odd_Even, Pin_Headers:Pin_Header_Straight_2x03_Pitch2.54mm, symbol Connector_Generic:Conn_02x03_Odd_Even
- added J4: Conn_01x04, Pin_Headers:Pin_Header_Straight_1x04_Pitch2.54mm, symbol Connector_Generic:Conn_01x04
- added J5: Conn_01x05, Pin_Headers:Pin_Header_Straight_1x05_Pitch2.54mm, symbol Connector_Generic:Conn_01x05
- added R1, R2, R3: 500 Ohm, Resistors_SMD:R_0805, symbol Device:R_US
Connections:
- new net: J4.1 (Pin_1), R1.1
- new net: J4.2 (Pin_2), R2.1
- new net: J4.3 (Pin_3), R3.1
- new net +3V3: J2.1 (Pin_1), J3.2 (Pin_2)
- new net GND: J2.2 (Pin_2), J3.1 (Pin_1), J4.4 (Pin_4), J5.5 (Pin_5)
- new net LCD_8BIT_0: J1.1 (Pin_1)
- new net LCD_8BIT_1: J1.3 (Pin_3)
- new net LCD_8BIT_2: J1.5 (Pin_5)
- new net LCD_8BIT_3: J1.7 (Pin_7)
- new net LCD_8BIT_4: J1.2 (Pin_2)
- new net LCD_8BIT_5: J1.4 (Pin_4)
- new net LCD_8BIT_6: J1.6 (Pin_6)
- new net LCD_8BIT_7: J1.8 (Pin_8)
- new net LCD_CCS: J2.7 (Pin_7)
- new net LCD_DC: J2.8 (Pin_8)
- new net LCD_MISO: J2.6 (Pin_6)
- new net LCD_MOSI: J2.5 (Pin_5)
- new net LCD_SCK: J2.3 (Pin_3)
- new net LCD_SEL: J2.4 (Pin_4)
- new net LCD_XM: J2.9 (Pin_9)
- new net LCD_XP: J2.11 (Pin_11)
- new net LCD_YM: J2.12 (Pin_12)
- new net LCD_YP: J2.10 (Pin_10)
- new net LED_GREEN: R3.2
- new net LED_RED: R1.2
- new net LED_YELLOW: R2.2
- new net NRST: J3.3 (Pin_3)
- new net SPARE_GPIO_0: J5.1 (Pin_1)
- new net SPARE_GPIO_1: J5.2 (Pin_2)
- new net SPARE_GPIO_2: J5.3 (Pin_3)
- new net SPARE_GPIO_3: J5.4 (Pin_4)
- new net SWCLK: J3.5 (Pin_5)
- new net SWDIO: J3.6 (Pin_6)
- no-connect marks 0 -> 1
Other:
- note added: "3V3"
- note added: "CCS"
- note added: "CS"
- note added: "Countdown LEDs"
- note added: "D/C | WR"
- note added: "GND"
- note added: "LCD 8-Bit header\n"
- note added: "LCD Header"
- note added: "MISO"
- note added: "MOSI | RD"
- note added: "Programming Header"
- note added: "SCK | C/D"
- note added: "Spare GPIO Header\n"
- note added: "X+"
- note added: "X-"
- note added: "Y+"
- note added: "Y-"
