File: hardware/remote_racing_pcb.kicad_pcb (KiCad board)
At the start: 2 copper layers, 110.5 x 41.9 mm, 35 parts, among them IC1 L86-M33, J1 Conn_02x04_Odd_Even, J2 Conn_01x12, J3 Conn_02x03_Odd_Even, J4 Conn_01x04, J5 Conn_01x05, U1 SparkFun_Pro_nRF52840_Mini, U2 STM32F030R8Tx

Commit message: PCB Layout Pre-Review
Parts:
- S1: value Reset -> Button
- TP11: renamed from GPS Force On
- TP13: renamed from IMU SCL
- TP15: renamed from IMU SDA
- TP2: renamed from GPS TX
- TP5: renamed from GPS RX
- TP8: renamed from GPS 1PPS
- moved C6 35.8 mm to (149.9, 98.2)
- moved AC1 35.8 mm to (158.8, 105.8)
- moved C1 35.8 mm to (153.3, 105.2)
- moved C10 35.8 mm to (140.6, 110.0)
- moved C11 35.8 mm to (151.1, 106.7)
- moved C2 35.8 mm to (155.2, 105.2)
- moved C4 35.8 mm to (120.1, 106.4)
- moved C5 35.8 mm to (118.0, 106.4)
- moved C8 35.8 mm to (140.6, 111.9)
- moved C9 35.8 mm to (149.2, 106.7)
- moved H3 35.8 mm to (121.9, 119.4)
- moved H4 35.8 mm to (191.8, 119.4)
- moved IC1 35.8 mm to (94.0, 104.1)
- moved J1 35.8 mm to (145.4, 86.4)
- moved J2 35.8 mm to (120.7, 88.9)
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Routing:
- net SPARE_GPIO_0: track 0.00 -> 15.0 mm
- net SPARE_GPIO_1: track 0.00 -> 14.2 mm
- net SPARE_GPIO_2: track 0.00 -> 13.4 mm
- net SPARE_GPIO_3: track 0.00 -> 12.5 mm
- net GND: track 31.6 -> 36.6 mm, vias 3 -> 5
- net IMU_SDA: track 41.2 -> 44.0 mm
- net +3V3: track 43.4 -> 46.0 mm
- net IMU_SCL: track 39.8 -> 42.1 mm
- added copper zone on B.Cu, net +3V3
- added copper zone on F.Cu, net GND
Other:
- rule trace_min: 0.2 -> 0.2032
- board text added: "0"
- board text added: "1"
- board text added: "2"
- board text added: "3"
- board text added: "3.3V"
- board text added: "4"
- board text added: "5"
- board text added: "6"
- board text added: "7"
- board text added: "CCS"
- board text added: "D/C (WR)"
- board text added: "GND"
- board text added: "Green"
- board text added: "MISO"
- board text added: "MOSI (RD)"
- board text added: "Red"
- board text added: "SCK (C/D)"
- board text added: "SEL"
- board text added: "X+"
- board text added: "X-"
- board text added: "Y+"
- board text added: "Y-"
- board text added: "Yellow"

Commit message: PCB Finished and Ordered
Parts:
- GPS 1PPS: renamed from TP8
- GPS FORCE ON: renamed from TP11
- GPS RX: renamed from TP5
- GPS TX: renamed from TP2
- IMU SCL: renamed from TP13
- IMU SDA: renamed from TP15
- LCD 8-bit: renamed from J4
- LCD SPI (8-bit): renamed from J2
- S1: value Button -> Reset
- Spare GPIO: renamed from J5
- renumbered J1 to LEDs, J3 to Program
Routing:
- net +3V3: track 46.0 -> 24.8 mm, vias 2 -> 1
Other:
- board text added: "NC"
- board text added: "NRST"
- board text added: "Remote Racing Device D. Salbert 2020-11-2"
- board text added: "SWCLK"
- board text added: "SWDIO"
Changed lines of the file:
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@@
   (general
     (thickness 1.6)
-    (drawings 39)
-    (tracks 322)
+    (drawings 46)
+    (tracks 313)
     (zones 0)
     (modules 35)
@@
     (descr "Through hole straight pin header, 2x04, 2.54mm pitch, double rows")
     (tags "Through hole pin header THT 2x04 2.54mm double row")
-    (fp_text reference J1 (at 0 -14.605 270 unlocked) (layer F.SilkS)
+    (fp_text reference LEDs (at 0 -14.605 270 unlocked) (layer F.SilkS)
       (effects (font (size 1 1) (thickness 0.15)))
     )
@@
     (descr "Through hole straight pin header, 1x05, 2.54mm pitch, single row")
     (tags "Through hole pin header THT 1x05 2.54mm single row")
-    (fp_text reference J5 (at -2.794 5.08 180) (layer F.SilkS)
+    (fp_text reference "Spare GPIO" (at -2.794 5.08 180) (layer F.SilkS)
       (effects (font (size 1 1) (thickness 0.15)))
     )
@@
     (descr "Keystone Miniature THM Test Point 5005-5009, http://www.keyelco.com/product-pdf.cfm?p=1314")
     (tags "Through Hole Mount Test Points")
-    (fp_text reference TP15 (at 0 2.794) (layer F.SilkS)
+    (fp_text reference "IMU SDA" (at 0 2.794) (layer F.SilkS)
       (effects (font (size 0.5 0.5) (thickness 0.125)))
     )
@@
     (descr "Keystone Miniature THM Test Point 5005-5009, http://www.keyelco.com/product-pdf.cfm?p=1314")
     (tags "Through Hole Mount Test Points")
-    (fp_text reference TP13 (at 0 2.794) (layer F.SilkS)
+    (fp_text reference "IMU SCL" (at 0 2.794) (layer F.SilkS)
       (effects (font (size 0.5 0.5) (thickness 0.125)))
     )
@@
     (descr "Keystone Miniature THM Test Point 5005-5009, http://www.keyelco.com/product-pdf.cfm?p=1314")
     (tags "Through Hole Mount Test Points")
-    (fp_text reference TP11 (at 0 -2.794 180 unlocked) (layer F.SilkS)
+    (fp_text reference "GPS FORCE ON" (at 0 -2.794 180 unlocked) (layer F.SilkS)
       (effects (font (size 0.5 0.5) (thickness 0.125)))
     )
@@
     (descr "Keystone Miniature THM Test Point 5005-5009, http://www.keyelco.com/product-pdf.cfm?p=1314")
     (tags "Through Hole Mount Test Points")
-    (fp_text reference TP8 (at -0.018 -2.794 180 unlocked) (layer F.SilkS)
+    (fp_text reference "GPS 1PPS" (at -0.018 -2.794 180 unlocked) (layer F.SilkS)
       (effects (font (size 0.5 0.5) (thickness 0.125)))
     )
@@
     (descr "Keystone Miniature THM Test Point 5005-5009, http://www.keyelco.com/product-pdf.cfm?p=1314")
     (tags "Through Hole Mount Test Points")
-    (fp_text reference TP5 (at 0 3.048) (layer F.SilkS)
+    (fp_text reference "GPS RX" (at 0 3.048) (layer F.SilkS)
       (effects (font (size 0.5 0.5) (thickness 0.125)))
     )
@@
     (descr "Keystone Miniature THM Test Point 5005-5009, http://www.keyelco.com/product-pdf.cfm?p=1314")
     (tags "Through Hole Mount Test Points")
-    (fp_text reference TP2 (at 0 3.139) (layer F.SilkS)
+    (fp_text reference "GPS TX" (at 0 3.139) (layer F.SilkS)
       (effects (font (size 0.5 0.5) (thickness 0.125)))
     )
@@
       (effects (font (size 1.27 1.27) (thickness 0.254)))
     )
-    (fp_text value Button (at 0.052 3.738) (layer F.SilkS)
+    (fp_text value Reset (at 0.052 3.738 180 unlocked) (layer F.SilkS)
       (effects (font (size 1.27 1.27) (thickness 0.254)))
     )
@@
     (descr "Through hole straight pin header, 1x04, 2.54mm pitch, single row")
     (tags "Through hole pin header THT 1x04 2.54mm single row")
-    (fp_text reference J4 (at -6.35 -8.509 180 unlocked) (layer F.SilkS)
+    (fp_text reference "LCD 8-bit" (at -6.35 -8.509 180 unlocked) (layer F.SilkS)
       (effects (font (size 1 1) (thickness 0.15)))
     )
@@
     (descr "Through hole straight pin header, 2x03, 2.54mm pitch, double rows")
     (tags "Through hole pin header THT 2x03 2.54mm double row")
-    (fp_text reference J3 (at 1.27 2.33) (layer B.SilkS)
-      (effects (font (size 1 1) (thickness 0.15)) (justify mirror))
+    (fp_text reference Program (at 1.27 2.794 180 unlocked) (layer F.SilkS)
+      (effects (font (size 1 1) (thickness 0.15)))
     )
     (fp_text value Conn_02x03_Odd_Even (at 1.27 -7.41) (layer B.Fab)
@@
     (descr "Through hole straight pin header, 2x06, 2.54mm pitch, double rows")
     (tags "Through hole pin header THT 2x06 2.54mm double row")
-    (fp_text reference J2 (at -4.826 6.35 180 unlocked) (layer F.SilkS)
+    (fp_text reference "LCD SPI (8-bit)" (at -4.826 6.35 180 unlocked) (layer F.SilkS)
       (effects (font (size 1 1) (thickness 0.15)))
     )
@@
     (tags "mounting hole 4.3mm no annular m4")
     (attr virtual)
-    (fp_text reference H4 (at 0 -5.3) (layer F.SilkS) hide
+    (fp_text reference H4 (at 0 5.08) (layer F.SilkS) hide
       (effects (font (size 1 1) (thickness 0.15)))
     )
@@
     (tags "mounting hole 4.3mm no annular m4")
     (attr virtual)
-    (fp_text reference H2 (at 0 -5.3) (layer F.SilkS)
+    (fp_text reference H2 (at 0 -5.3) (layer F.SilkS) hide
       (effects (font (size 1 1) (thickness 0.15)))
     )
@@
     (tags "capacitor 0805")
     (attr smd)
-    (fp_text reference C6 (at 0 -1.5 270) (layer F.SilkS)
+    (fp_text reference C6 (at 2.54 0 180 unlocked) (layer F.SilkS)
       (effects (font (size 1 1) (thickness 0.15)))
     )
@@
     )
   )
+  (gr_text GND (at 159.131 99.568 180) (layer F.SilkS)
+    (effects (font (size 0.5 0.5) (thickness 0.125)))
+  )
+  (gr_text NRST (at 159.004 97.028 180) (layer F.SilkS)
+    (effects (font (size 0.5 0.5) (thickness 0.125)))
+  )
+  (gr_text NC (at 161.29 97.028 180) (layer F.SilkS)
+    (effects (font (size 0.5 0.5) (thickness 0.125)))
+  )
+  (gr_text SWCLK (at 158.75 94.488 180) (layer F.SilkS)
+    (effects (font (size 0.5 0.5) (thickness 0.125)))
+  )
+  (gr_text SWDIO (at 161.925 94.488 180) (layer F.SilkS)
+    (effects (font (size 0.5 0.5) (thickness 0.125)))
+  )
+  (gr_text 3.3V (at 161.671 99.568 180) (layer F.SilkS)
+    (effects (font (size 0.5 0.5) (thickness 0.125)))
+  )
+  (gr_text "Remote Racing Device\nD. Salbert 2020-11-2" (at 192.405 103.505 90) (layer F.SilkS)
+    (effects (font (size 1 1) (thickness 0.15)))
+  )
   (gr_text 3.3V (at 120.65 91.186 180) (layer F.SilkS)
     (effects (font (size 0.5 0.5) (thickness 0.125)))
@@
   (segment (start 139.355 109.748) (end 139.589 109.982) (width 0.25) (layer B.Cu) (net 3))
   (segment (start 139.355 107.985) (end 139.355 109.748) (width 0.25) (layer B.Cu) (net 3))
-  (segment (start 135.855 98.485) (end 135.855 97.882) (width 0.25) (layer B.Cu) (net 3))
-  (segment (start 134.604 96.663) (end 133.985 96.663) (width 0.25) (layer B.Cu) (net 3))
-  (segment (start 135.855 97.658) (end 135.855 97.882) (width 0.25) (layer B.Cu) (net 3))
-  (segment (start 134.86 96.663) (end 135.855 97.658) (width 0.25) (layer B.Cu) (net 3))
-  (segment (start 133.985 96.663) (end 134.86 96.663) (width 0.25) (layer B.Cu) (net 3))
   (segment (start 159.25 108.926) (end 159.29 108.966) (width 0.25) (layer B.Cu) (net 3))
   (segment (start 159.25 107.066) (end 159.25 108.926) (width 0.25) (layer B.Cu) (net 3))
-  (segment (start 120.65 90) (end 120.82 90.17) (width 0.25) (layer F.Cu) (net 3))
-  (segment (start 120.65 88.9) (end 120.65 90) (width 0.25) (layer F.Cu) (net 3))
-  (segment (start 120.82 90.17) (end 133.35 90.17) (width 0.25) (layer F.Cu) (net 3))
-  (via (at 134.075 95.25) (size 0.8) (drill 0.4) (layers F.Cu B.Cu) (net 3))
-  (segment (start 133.35 90.17) (end 134.075 90.895) (width 0.25) (layer F.Cu) (net 3))
-  (segment (start 134.075 90.895) (end 134.075 95.25) (width 0.25) (layer F.Cu) (net 3))
-  (segment (start 134.075 96.573) (end 133.985 96.663) (width 0.25) (layer B.Cu) (net 3))
-  (segment (start 134.075 95.25) (end 134.075 96.573) (width 0.25) (layer B.Cu) (net 3))
   (segment (start 109.48 107.2) (end 109.48 105.41) (width 0.25) (layer F.Cu) (net 3))
   (segment (start 109.48 107.95) (end 109.48 107.2) (width 0.25) (layer F.Cu) (net 3))
@@
   (segment (start 145.355 107.985) (end 146.015 107.985) (width 0.25) (layer B.Cu) (net 3))
   (segment (start 147.355 105.985) (end 147.355 106.645) (width 0.25) (layer B.Cu) (net 3))
+  (segment (start 135.855 98.085) (end 135.855 98.485) (width 0.25) (layer B.Cu) (net 3))
+  (segment (start 135.855 97.610304) (end 135.855 98.085) (width 0.25) (layer B.Cu) (net 3))
+  (segment (start 134.907696 96.663) (end 135.855 97.610304) (width 0.25) (layer B.Cu) (net 3))
+  (segment (start 133.985 96.663) (end 134.907696 96.663) (width 0.25) (layer B.Cu) (net 3))
   (via (at 161.036 105.41) (size 0.8) (drill 0.4) (layers F.Cu B.Cu) (net 5))
   (segment (start 160.025 105.791) (end 160.655 105.791) (width 0.25) (layer B.Cu) (net 5))
