File: hardware/IMU.sch (KiCad schematic (older format))
At the start: 4 parts

Commit message: Pcb development (#1)
* PCB Finished and Ordered
Parts:
- added R4: 10k, Resistors_SMD:R_0805, symbol Device:R_US
- AC1: renamed from AC?; footprint MMA8452QR1 -> Mouser_Components:MMA8452QR1
- C1, C2, C3: renamed from C?; footprint (none) -> Capacitors_SMD:C_0805
Connections:
- net +3V3: now also R4.1
- net GND: now also AC1.10 (GND_2), AC1.12 (GND_3), C3.2
- net IMU_INT_1: now reaches AC1.11 (INT1)
- net at AC1.7 (SA0): now also R4.2
- net IMU_INT_2: now reaches AC1.9 (INT2)
- net accel_SCL renamed IMU_SCL
- net accel_SDA renamed IMU_SDA
Other:
- note added: "SAO = 1:\nI2C Address = 0x1D"
- moved on the sheet: AC1, C1, C2, C3
Changed lines of the file:
@@
 $Descr A4 11693 8268
 encoding utf-8
-Sheet 5 8
+Sheet 5 7
 Title ""
 Date ""
@@
 Comment4 ""
 $EndDescr
-Text GLabel 5400 4600 0    50   Input ~ 0
-accel_SCL
-Text GLabel 5900 5300 3    50   Input ~ 0
-accel_SDA
+Text GLabel 5350 4150 0    50   Input ~ 0
+IMU_SCL
+Text GLabel 5850 4850 3    50   Input ~ 0
+IMU_SDA
 Wire Wire Line
-	6600 4400 6850 4400
+	6550 3950 6800 3950
 $Comp
-L Device:C C?
+L Device:C C3
 U 1 1 5F9263CF
-P 6850 4050
-F 0 "C?" H 6965 4096 50  0000 L CNN
-F 1 "4.7uF" H 6965 4005 50  0000 L CNN
-F 2 "" H 6888 3900 50  0001 C CNN
-F 3 "~" H 6850 4050 50  0001 C CNN
-	1    6850 4050
+P 6800 3600
+F 0 "C3" H 6915 3646 50  0000 L CNN
+F 1 "4.7uF" H 6915 3555 50  0000 L CNN
+F 2 "Capacitors_SMD:C_0805" H 6838 3450 50  0001 C CNN
+F 3 "~" H 6800 3600 50  0001 C CNN
+	1    6800 3600
 	1    0    0    -1
 $EndComp
 Wire Wire Line
-	6850 3700 6100 3700
-Text Notes 6900 3900 0    50   ~ 0
+	6800 3250 6050 3250
+Text Notes 6850 3450 0    50   ~ 0
 Place Ceramic \nCapacitor near pins
 Wire Wire Line
-	6850 3700 6850 3900
+	6800 3250 6800 3450
 Wire Wire Line
-	6850 4200 6850 4400
+	6800 3750 6800 3950
 $Comp
-L Mouser_Components:MMA8452QR1 AC?
+L Mouser_Components:MMA8452QR1 AC1
 U 1 1 5F92167B
-P 5400 4300
-F 0 "AC?" H 6000 5081 50  0000 C CNN
-F 1 "MMA8452QR1" H 6000 4990 50  0000 C CNN
-F 2 "MMA8452QR1" H 6450 4700 50  0001 L CNN
-F 3 "http://www.nxp.com/docs/en/data-sheet/MMA8452Q.pdf" H 6450 4600 50  0001 L CNN
-F 4 "NXP - MMA8452QR1 - ACCELEROMETER, 1024/512/256COUNTS/G, QFN" H 6450 4500 50  0001 L CNN "Description"
-F 5 "1" H 6450 4400 50  0001 L CNN "Height"
-F 6 "841-MMA8452QR1" H 6450 4300 50  0001 L CNN "Mouser Part Number"
-F 7 "https://www.mouser.co.uk/ProductDetail/NXP-Semiconductors/MMA8452QR1?qs=nf24X8JpkflP9lEXYucw7A%3D%3D" H 6450 4200 50  0001 L CNN "Mouser Price/Stock"
-F 8 "NXP" H 6450 4100 50  0001 L CNN "Manufacturer_Name"
-F 9 "MMA8452QR1" H 6450 4000 50  0001 L CNN "Manufacturer_Part_Number"
-	1    5400 4300
+P 5350 3850
+F 0 "AC1" H 5950 4631 50  0000 C CNN
+F 1 "MMA8452QR1" H 5950 4540 50  0000 C CNN
+F 2 "Mouser_Components:MMA8452QR1" H 6400 4250 50  0001 L CNN
+F 3 "http://www.nxp.com/docs/en/data-sheet/MMA8452Q.pdf" H 6400 4150 50  0001 L CNN
+F 4 "NXP - MMA8452QR1 - ACCELEROMETER, 1024/512/256COUNTS/G, QFN" H 6400 4050 50  0001 L CNN "Description"
+F 5 "1" H 6400 3950 50  0001 L CNN "Height"
+F 6 "841-MMA8452QR1" H 6400 3850 50  0001 L CNN "Mouser Part Number"
+F 7 "https://www.mouser.co.uk/ProductDetail/NXP-Semiconductors/MMA8452QR1?qs=nf24X8JpkflP9lEXYucw7A%3D%3D" H 6400 3750 50  0001 L CNN "Mouser Price/Stock"
+F 8 "NXP" H 6400 3650 50  0001 L CNN "Manufacturer_Name"
+F 9 "MMA8452QR1" H 6400 3550 50  0001 L CNN "Manufacturer_Part_Number"
+	1    5350 3850
 	1    0    0    -1
 $EndComp
-NoConn ~ 5900 3700
-NoConn ~ 6000 3700
-NoConn ~ 6100 5300
-NoConn ~ 6600 4300
+NoConn ~ 5850 3250
+NoConn ~ 5950 3250
+NoConn ~ 6050 4850
+NoConn ~ 6550 3850
 $Comp
-L power:+3.3V #PWR?
+L power:+3.3V #PWR0117
 U 1 1 5F92A081
-P 6850 3700
-F 0 "#PWR?" H 6850 3550 50  0001 C CNN
-F 1 "+3.3V" H 6865 3873 50  0000 C CNN
-F 2 "" H 6850 3700 50  0001 C CNN
-F 3 "" H 6850 3700 50  0001 C CNN
-	1    6850 3700
+P 6800 3250
+F 0 "#PWR0117" H 6800 3100 50  0001 C CNN
+F 1 "+3.3V" H 6815 3423 50  0000 C CNN
+F 2 "" H 6800 3250 50  0001 C CNN
+F 3 "" H 6800 3250 50  0001 C CNN
+	1    6800 3250
 	1    0    0    -1
 $EndComp
-Connection ~ 6850 3700
+Connection ~ 6800 3250
 $Comp
-L power:+3.3V #PWR?
+L power:+3.3V #PWR0118
 U 1 1 5F92B3EA
-P 4000 4300
-F 0 "#PWR?" H 4000 4150 50  0001 C CNN
-F 1 "+3.3V" H 4015 4473 50  0000 C CNN
-F 2 "" H 4000 4300 50  0001 C CNN
-F 3 "" H 4000 4300 50  0001 C CNN
-	1    4000 4300
+P 3950 3850
+F 0 "#PWR0118" H 3950 3700 50  0001 C CNN
+F 1 "+3.3V" H 3965 4023 50  0000 C CNN
+F 2 "" H 3950 3850 50  0001 C CNN
+F 3 "" H 3950 3850 50  0001 C CNN
+	1    3950 3850
 	1    0    0    -1
 $EndComp
-NoConn ~ 5400 4500
+NoConn ~ 5350 4050
 $Comp
-L Device:C C?
+L Device:C C2
 U 1 1 5F92D4E8
-P 4500 4550
-F 0 "C?" H 4615 4596 50  0000 L CNN
-F 1 "0.1nF" H 4615 4505 50  0000 L CNN
-F 2 "" H 4538 4400 50  0001 C CNN
-F 3 "~" H 4500 4550 50  0001 C CNN
-	1    4500 4550
+P 4450 4100
+F 0 "C2" H 4565 4146 50  0000 L CNN
+F 1 "0.1nF" H 4565 4055 50  0000 L CNN
+F 2 "Capacitors_SMD:C_0805" H 4488 3950 50  0001 C CNN
+F 3 "~" H 4450 4100 50  0001 C CNN
+	1    4450 4100
 	1    0    0    -1
 $EndComp
 Wire Wire Line
-	5400 4400 4500 4400
+	5350 3950 4450 3950
 $Comp
-L Device:C C?
+L Device:C C1
 U 1 1 5F92E7E2
-P 4000 4550
-F 0 "C?" H 4115 4596 50  0000 L CNN
-F 1 "0.1nF" H 4115 4505 50  0000 L CNN
-F 2 "" H 4038 4400 50  0001 C CNN
-F 3 "~" H 4000 4550 50  0001 C CNN
-	1    4000 4550
+P 3950 4100
+F 0 "C1" H 4065 4146 50  0000 L CNN
+F 1 "0.1nF" H 4065 4055 50  0000 L CNN
+F 2 "Capacitors_SMD:C_0805" H 3988 3950 50  0001 C CNN
+F 3 "~" H 3950 4100 50  0001 C CNN
+	1    3950 4100
 	1    0    0    -1
 $EndComp
 Wire Wire Line
-	5400 4300 4000 4300
+	5350 3850 3950 3850
 Wire Wire Line
-	4000 4300 4000 4400
-Connection ~ 4000 4300
+	3950 3850 3950 3950
+Connection ~ 3950 3850
 Wire Wire Line
-	4000 4700 4500 4700
+	3950 4250 4450 4250
 Wire Wire Line
-	4500 4700 5400 4700
-Connection ~ 4500 4700
+	4450 4250 5350 4250
+Connection ~ 4450 4250
 $Comp
-L power:GND #PWR?
+L power:GND #PWR0119
 U 1 1 5F930686
-P 4000 4700
-F 0 "#PWR?" H 4000 4450 50  0001 C CNN
-F 1 "GND" H 4005 4527 50  0000 C CNN
-F 2 "" H 4000 4700 50  0001 C CNN
-F 3 "" H 4000 4700 50  0001 C CNN
-	1    4000 4700
+P 3950 4250
+F 0 "#PWR0119" H 3950 4000 50  0001 C CNN
+F 1 "GND" H 3955 4077 50  0000 C CNN
+F 2 "" H 3950 4250 50  0001 C CNN
+F 3 "" H 3950 4250 50  0001 C CNN
+	1    3950 4250
 	1    0    0    -1
 $EndComp
-Connection ~ 4000 4700
+Connection ~ 3950 4250
+$Comp
+L power:GND #PWR0120
+U 1 1 5F924880
+P 7200 4250
+F 0 "#PWR0120" H 7200 4000 50  0001 C CNN
+F 1 "GND" H 7205 4077 50  0000 C CNN
+F 2 "" H 7200 4250 50  0001 C CNN
+F 3 "" H 7200 4250 50  0001 C CNN
+	1    7200 4250
+	1    0    0    -1
+$EndComp
+Wire Wire Line
+	7200 4150 7200 4250
+Wire Wire Line
+	5950 4850 5950 5000
+$Comp
+L power:+3.3V #PWR0121
+U 1 1 5F9274C7
+P 6800 5000
+F 0 "#PWR0121" H 6800 4850 50  0001 C CNN
+F 1 "+3.3V" V 6800 5250 50  0000 C CNN
+F 2 "" H 6800 5000 50  0001 C CNN
+F 3 "" H 6800 5000 50  0001 C CNN
+	1    6800 5000
+	0    1    1    0
+$EndComp
+Wire Wire Line
+	5950 5000 6500 5000
+$Comp
+L Device:R_US R4
+U 1 1 5F92A823
+P 6650 5000
+F 0 "R4" V 6445 5000 50  0000 C CNN
+F 1 "10k" V 6536 5000 50  0000 C CNN
+F 2 "Resistors_SMD:R_0805" V 6690 4990 50  0001 C CNN
+F 3 "~" H 6650 5000 50  0001 C CNN
+	1    6650 5000
+	0    1    1    0
+$EndComp
+Text Notes 6350 5250 0    50   ~ 0
+SAO = 1:\nI2C Address = 0x1D
+Text GLabel 6550 4050 2    50   Input ~ 0
+IMU_INT_1
+Text GLabel 6550 4250 2    50   Input ~ 0
+IMU_INT_2
+Wire Wire Line
+	6550 4150 7200 4150
+Wire Wire Line
+	6800 3950 7200 3950
+Wire Wire Line
+	7200 3950 7200 4150
+Connection ~ 6800 3950
+Connection ~ 7200 4150
 $EndSCHEMATC
