File: hardware/Microcontroller.sch (KiCad schematic (older format))
At the start: 6 parts

Commit message: Pcb development (#1)
* PCB Finished and Ordered
Parts:
- added C6: 100nF, Capacitors_SMD:C_0805, symbol Device:C
- added S1: Button, SKQGAKE010, symbol Mouser_Components:SKQGAKE010
- C10, C11, C7, C8, C9: renamed from C?; footprint (none) -> Capacitors_SMD:C_0805
- U2: renamed from U?; footprint Package_QFP:LQFP-64_10x10mm_P0.5mm -> Digikey Library:64-LQFP_(10x10)
Connections:
- net GND: now also U2.60 (BOOT0), C6.2, S1.4
- net GPS_1PPS: now reaches U2.14 (PA0)
- net GPS_FORCE_ON: now reaches U2.15 (PA1)
- net GPS_RX: now reaches U2.16 (PA2)
- net GPS_TX: now reaches U2.17 (PA3)
- net SPARE_GPIO_0: now reaches U2.2 (PC13)
- net LCD_SEL: now reaches U2.20 (PA4)
- net LCD_SCK: now reaches U2.21 (PA5)
- net LCD_MISO: now reaches U2.22 (PA6)
- net LCD_MOSI: now reaches U2.23 (PA7)
- net LCD_DC: now reaches U2.24 (PC4)
- net LCD_CCS: now reaches U2.25 (PC5)
- net LCD_YP: now reaches U2.26 (PB0)
- net LCD_XM: now reaches U2.27 (PB1)
- net LCD_YM: now reaches U2.28 (PB2)
- net LCD_XP: now reaches U2.29 (PB10)
- net SPARE_GPIO_1: now reaches U2.3 (PC14)
- net LCD_8BIT_3: now reaches U2.33 (PB12)
- net LCD_8BIT_7: now reaches U2.34 (PB13)
- net LCD_8BIT_2: now reaches U2.35 (PB14)
- net LCD_8BIT_6: now reaches U2.36 (PB15)
- net LCD_8BIT_1: now reaches U2.37 (PC6)
- net LCD_8BIT_5: now reaches U2.38 (PC7)
- net LCD_8BIT_0: now reaches U2.39 (PC8)
- net SPARE_GPIO_2: now reaches U2.4 (PC15)
- net LCD_8BIT_4: now reaches U2.40 (PC9)
- net BLE_RX: now reaches U2.42 (PA9)
- net BLE_TX: now reaches U2.43 (PA10)
- net SWDIO: now reaches U2.46 (PA13)
- net SWCLK: now reaches U2.49 (PA14)
- net SPARE_GPIO_3: now reaches U2.5 (PF0)
- net LED_GREEN: now reaches U2.50 (PA15)
- net LED_YELLOW: now reaches U2.51 (PC10)
- net LED_RED: now reaches U2.52 (PC11)
- net IMU_INT_2: now reaches U2.57 (PB5)
- net IMU_INT_1: now reaches U2.58 (PB6)
- net NRST: now reaches U2.7 (NRST)
- net NRST: now also C6.1, S1.2
- net accel_SCL renamed IMU_SCL
- net accel_SDA renamed IMU_SDA
- no-connect marks 0 -> 20
Other:
- note added: "Reset Button"
- moved on the sheet: C10, C11, C7, C8, C9, U2
