File: hardware/Power.sch (KiCad schematic (older format))
At the start: 0 parts

Commit message: Pcb development (#1)
* PCB Finished and Ordered
Parts:
- added C? (x2): 1uF, symbol Device:C
- added IC?: NCP164CSN330T1G, SOT95P275X110-5N, symbol Mouser_Components:NCP164CSN330T1G
- added IC?: L6924D013TR, QFN50P300X300X100-17N-D, symbol Mouser_Components:L6924D013TR
Connections:
- net labels added: +3.3V, +BATT, GND
- wire segments 0 -> 8
- no-connect marks 0 -> 1
Other:
- note added: "3.3V Regulator\nUse Ceramic Caps"
- note added: "Battery Charging"
- note added: "Dropout voltage: 110mV at 300mA\n(3.41V)"
Changed lines of the file:
@@
 Comment4 ""
 $EndDescr
+$Comp
+L Mouser_Components:NCP164CSN330T1G IC?
+U 1 1 5F97A251
+P 8400 3500
+F 0 "IC?" H 9000 3765 50  0000 C CNN
+F 1 "NCP164CSN330T1G" H 9000 3674 50  0000 C CNN
+F 2 "SOT95P275X110-5N" H 9450 3600 50  0001 L CNN
+F 3 "https://componentsearchengine.com/Datasheets/2/NCP164CSN330T1G.pdf" H 9450 3500 50  0001 L CNN
+F 4 "LDO Regulator Pos 3.3V 0.3A 5-Pin TSOP T/R" H 9450 3400 50  0001 L CNN "Description"
+F 5 "1.1" H 9450 3300 50  0001 L CNN "Height"
+F 6 "863-NCP164CSN330T1G" H 9450 3200 50  0001 L CNN "Mouser Part Number"
+F 7 "https://www.mouser.co.uk/ProductDetail/ON-Semiconductor/NCP164CSN330T1G?qs=xZ%2FP%252Ba9zWqbi%2FAyy5UtoRw%3D%3D" H 9450 3100 50  0001 L CNN "Mouser Price/Stock"
+F 8 "ON Semiconductor" H 9450 3000 50  0001 L CNN "Manufacturer_Name"
+F 9 "NCP164CSN330T1G" H 9450 2900 50  0001 L CNN "Manufacturer_Part_Number"
+	1    8400 3500
+	1    0    0    -1
+$EndComp
+Text Notes 8650 3100 0    50   ~ 0
+  3.3V Regulator\nUse Ceramic Caps
+$Comp
+L power:GND #PWR?
+U 1 1 5F96BE1C
+P 9800 3900
+F 0 "#PWR?" H 9800 3650 50  0001 C CNN
+F 1 "GND" H 9805 3727 50  0000 C CNN
+F 2 "" H 9800 3900 50  0001 C CNN
+F 3 "" H 9800 3900 50  0001 C CNN
+	1    9800 3900
+	1    0    0    -1
+$EndComp
+$Comp
+L Device:C C?
+U 1 1 5F96AED7
+P 9800 3750
+F 0 "C?" H 9915 3796 50  0000 L CNN
+F 1 "1uF" H 9915 3705 50  0000 L CNN
+F 2 "" H 9838 3600 50  0001 C CNN
+F 3 "~" H 9800 3750 50  0001 C CNN
+	1    9800 3750
+	1    0    0    -1
+$EndComp
+$Comp
+L power:+3.3V #PWR?
+U 1 1 5F967017
+P 9800 3600
+F 0 "#PWR?" H 9800 3450 50  0001 C CNN
+F 1 "+3.3V" H 9815 3773 50  0000 C CNN
+F 2 "" H 9800 3600 50  0001 C CNN
+F 3 "" H 9800 3600 50  0001 C CNN
+	1    9800 3600
+	1    0    0    -1
+$EndComp
+$Comp
+L Device:C C?
+U 1 1 5F9636FB
+P 7850 3650
+F 0 "C?" H 7965 3696 50  0000 L CNN
+F 1 "1uF" H 7965 3605 50  0000 L CNN
+F 2 "" H 7888 3500 50  0001 C CNN
+F 3 "~" H 7850 3650 50  0001 C CNN
+	1    7850 3650
+	1    0    0    -1
+$EndComp
+$Comp
+L power:+BATT #PWR?
+U 1 1 5F961ABE
+P 7850 3500
+F 0 "#PWR?" H 7850 3350 50  0001 C CNN
+F 1 "+BATT" H 7865 3673 50  0000 C CNN
+F 2 "" H 7850 3500 50  0001 C CNN
+F 3 "" H 7850 3500 50  0001 C CNN
+	1    7850 3500
+	1    0    0    -1
+$EndComp
+Wire Wire Line
+	7850 3500 8300 3500
+Wire Wire Line
+	8400 3600 8200 3600
+Wire Wire Line
+	8200 3600 8200 3800
+Wire Wire Line
+	8200 3800 7850 3800
+Connection ~ 7850 3500
+Wire Wire Line
+	9600 3600 9800 3600
+Connection ~ 9800 3600
+Wire Wire Line
+	8400 3700 8300 3700
+Wire Wire Line
+	8300 3700 8300 3500
+Connection ~ 8300 3500
+Wire Wire Line
+	8300 3500 8400 3500
+$Comp
+L power:GND #PWR?
+U 1 1 5F9845B0
+P 7850 3800
+F 0 "#PWR?" H 7850 3550 50  0001 C CNN
+F 1 "GND" H 7855 3627 50  0000 C CNN
+F 2 "" H 7850 3800 50  0001 C CNN
+F 3 "" H 7850 3800 50  0001 C CNN
+	1    7850 3800
+	1    0    0    -1
+$EndComp
+Connection ~ 7850 3800
+NoConn ~ 9600 3500
+Text Notes 8250 4150 0    50   ~ 0
+Dropout voltage: 110mV at 300mA\n(3.41V)
+Text Notes 2050 3000 0    50   ~ 0
+Battery Charging
+$Comp
+L Mouser_Components:L6924D013TR IC?
+U 1 1 5FA0FE9F
+P 2150 4300
+F 0 "IC?" H 3594 4196 50  0000 L CNN
+F 1 "L6924D013TR" H 3594 4105 50  0000 L CNN
+F 2 "QFN50P300X300X100-17N-D" H 3400 4700 50  0001 L CNN
+F 3 "http://www.st.com/content/ccc/resource/technical/document/datasheet/group2/50/c4/60/ab/e6/09/4f/80/CD00079821/files/CD00079821.pdf/jcr:content/translations/en.CD00079821.pdf" H 3400 4600 50  0001 L CNN
+F 4 "STMICROELECTRONICS - L6924D013TR - QFN 16/BATTERY CHARGER SYSTEM" H 3400 4500 50  0001 L CNN "Description"
+F 5 "1" H 3400 4400 50  0001 L CNN "Height"
+F 6 "511-L6924D013TR" H 3400 4300 50  0001 L CNN "Mouser Part Number"
+F 7 "https://www.mouser.co.uk/ProductDetail/STMicroelectronics/L6924D013TR?qs=sZ9INdjBHvd2z7dh9ZwpeQ%3D%3D" H 3400 4200 50  0001 L CNN "Mouser Price/Stock"
+F 8 "STMicroelectronics" H 3400 4100 50  0001 L CNN "Manufacturer_Name"
+F 9 "L6924D013TR" H 3400 4000 50  0001 L CNN "Manufacturer_Part_Number"
+	1    2150 4300
+	1    0    0    -1
+$EndComp
 $EndSCHEMATC
