File: hardware/remote_racing_pcb.sch (KiCad schematic (older format))
At the start: 0 parts

Commit message: Pcb development (#1)
* PCB Finished and Ordered
Changed lines of the file:
@@
 $Descr A4 11693 8268
 encoding utf-8
-Sheet 1 8
+Sheet 1 7
 Title ""
 Date ""
@@
 $EndDescr
 $Sheet
-S 1500 3500 1500 1000
-U 5F8FB327
-F0 "Microcontroller" 50
-F1 "Microcontroller.sch" 50
+S 4000 5500 1500 1000
+U 5F96E2E5
+F0 "Misc" 50
+F1 "Misc.sch" 50
 $EndSheet
 $Sheet
-S 1500 1500 1500 1000
-U 5F8FBA81
-F0 "Power" 50
-F1 "Power.sch" 50
+S 4000 3500 1500 1000
+U 5F9239BE
+F0 "IO" 50
+F1 "IO.sch" 50
+$EndSheet
+$Sheet
+S 1500 3500 1500 1000
+U 5F923853
+F0 "Bluetooth" 50
+F1 "Bluetooth.sch" 50
+$EndSheet
+$Sheet
+S 4000 1500 1500 1000
+U 5F9237A0
+F0 "IMU" 50
+F1 "IMU.sch" 50
 $EndSheet
 $Sheet
@@
 $EndSheet
 $Sheet
-S 4000 1500 1500 1000
-U 5F9237A0
-F0 "IMU" 50
-F1 "IMU.sch" 50
-$EndSheet
-$Sheet
-S 4000 3500 1500 1000
-U 5F923853
-F0 "Bluetooth" 50
-F1 "Bluetooth.sch" 50
-$EndSheet
-$Sheet
-S 4000 5500 1500 1000
-U 5F923907
-F0 "LCD" 50
-F1 "LCD.sch" 50
-$EndSheet
-$Sheet
-S 6500 1500 1500 1000
-U 5F9239BE
-F0 "IO" 50
-F1 "IO.sch" 50
+S 1500 1500 1500 1000
+U 5F8FB327
+F0 "Microcontroller" 50
+F1 "Microcontroller.sch" 50
 $EndSheet
 $EndSCHEMATC
